Commit message: Implementing force drive that reacts to obstacles

File: mycode/drone_description/urdf/X500V2.urdf.xacro (robot description, xacro)
@@ -7,5 +7,5 @@
   <xacro:property name="robot_color" value="$(arg color)"/>
   <!-- Collision model dimensions (meters) -->
-  <xacro:property name="base_collision_radius" value="0.28"/>
+  <xacro:property name="base_collision_radius" value="0.45"/>
   <xacro:property name="base_collision_height" value="0.36"/>
   <xacro:property name="prop_collision_radius" value="0.13"/>
@@ -63,5 +63,5 @@
       </geometry>
     </collision>
-    <xacro:property name="prop_z" value="${-base_collision_height/2.0 + prop_centroid_z}"/>
+    <!-- <xacro:property name="prop_z" value="${-base_collision_height/2.0 + prop_centroid_z}"/>
     <collision name="prop_collision_front_left">
       <origin xyz="${prop_diag_offset} ${prop_diag_offset} ${prop_z}" rpy="0 0 0"/>
@@ -87,5 +87,5 @@
         <cylinder radius="${prop_collision_radius}" length="${prop_collision_height}"/>
       </geometry>
-    </collision>
+    </collision> -->
     <inertial>
       <origin xyz="0 0 0" rpy="0 0 0"/>

Commit message: Using repulsion proportionate to dist square

File: mycode/drone_description/urdf/X500V2.urdf.xacro (robot description, xacro)
@@ -37,5 +37,5 @@
         <box size="0.08 0.04 0.01"/>
       </geometry>
-      <material name="blue"/>
+      <material name="${robot_color}"/>
     </visual>
   </link>
